File: pcb/puggle.kicad_pcb (KiCad board)
At the start: 2 copper layers, 121 x 106.2 mm, 48 parts, among them J2 4PIN, SW1 SW_PUSH, SW10 SW_PUSH, SW11 SW_PUSH, SW12 SW_PUSH, SW13 SW_PUSH, SW14 SW_PUSH, SW15 SW_PUSH, SW16 SW_PUSH, SW17 SW_PUSH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

Commit message: Minor changes prior to prototype production.
Routing:
- net row3: track 157.2 -> 149.4 mm
- net row2: track 123.3 -> 122.7 mm
